File: Controller.kicad_pcb (KiCad board)
At the start: 6 copper layers, 50 x 50 mm, 197 parts, among them J201 U.FL-R-SMT-1, J801 HC-TYPE-C-16P-026W, J901 FPC-0.5AL-12PB, J902 FPC-0.5AL-12PB, J903 FPC-0.5AL-12PB, J904 FPC-0.5AL-12PB, J905 FPC-0.5AL-12PB, J906 FPC-0.5AL-12PB, Q301 30P03D, Q302 2N7002KNC, Q303 2N7002KNC, Q304 2N7002KNC, Q306 2N7002KNC, Q401 2N7002KNC, Q402 2N7002KNC, Q501 SI8487DB, Q502 SI8487DB, Q503 BSC0805LS, SW201 TSA016, U101 TXS0102, U201 ESP32-C3, U202 ZD25WQ32C, U203 WS2816C-1313, U301 SIC431A, U302 DZDH0401DW, U303 AP62600, U304 SY8301, U306 LMV331, U501 LP8866, U601 AL1793, U701 AL1793, U702 AL1793, U801 CH221K, Y201 2.D.1.400000920 40MHz

Commit message: Add files via upload
Parts:
- removed C203, C205, C207: 1u, Perfect passives:C 0402 (1005 Metric)
- removed C204, C210, C211: 100n, Perfect passives:C 0402 (1005 Metric)
- removed C206: 10n, Perfect passives:C 0402 (1005 Metric)
- removed C208, C209: TDB, Perfect passives:C 0402 (1005 Metric)
- removed C212, C213: 12p, Perfect passives:C 0402 (1005 Metric)
- removed C316: 10u, Perfect passives:C 0805 (2012 Metric)
- removed D202: LEDR, LED SMD:LED-0402-R
- removed D309: LESD8D3.3CAT5G, DFN-x:DFN-1006-2L
- removed JP502: Conn_02x03_Odd_Even, Connector_PinHeader_1.00mm:PinHeader_2x03_P1.00mm_Vertical
- removed JP801: Jumper_2_Small_Open, Solder jumpers:Jumper-NO 2P (1.9x1.4)
- removed L201: 2n, Perfect passives:L 0402 (1005 Metric)
- removed L202: TBD, Perfect passives:L 0402 (1005 Metric)
- removed L203: 24n, Perfect passives:L 0402 (1005 Metric)
- removed Q302: 2N7002KNC, DFN-x:DFN-1006-3L
- removed R205, R802: 1k, Perfect passives:R 0402 (1005 Metric)
- removed R321, R322: 121k, Perfect passives:R 0402 (1005 Metric)
- removed R324: 100k, Perfect passives:R 0402 (1005 Metric)
- removed R325: 6k, Perfect passives:R 0402 (1005 Metric)
- removed R327: 20k, Perfect passives:R 0402 (1005 Metric)
- removed R514: 11k, Perfect passives:R 0402 (1005 Metric)
- removed R801: 200k, Perfect passives:R 0402 (1005 Metric)
- removed SW201: TSA016, Buttons SMD:TSA016
- removed U306: LMV331, SOT-xxx:SOT-363-5
- removed U801: CH221K, SOT-xxx:SOT-23-6
- removed Y201: 2.D.1.400000920 40MHz, Crystals SMD:SMD-2016-4P
- added C214: 10u, Perfect passives:C 0805 (2012 Metric), F.Cu at (163.0, 106.2)
- added C215: 100n, Perfect passives:C 0402 (1005 Metric), F.Cu at (162.2, 99.5)
- added C518: 10u, Perfect passives:C 0805 (2012 Metric), F.Cu at (127.5, 76.8)
- added C519: 22u, Capacitor_SMD:C_1206_3216Metric, F.Cu at (129.8, 77.5)
- added C520: 10u, Perfect passives:C 0805 (2012 Metric), F.Cu at (117.0, 88.8)
- added C521: 10u, Perfect passives:C 0805 (2012 Metric), F.Cu at (117.0, 90.8)
- added C522: 10u, Perfect passives:C 0805 (2012 Metric), F.Cu at (117.0, 92.8)
- added C803: 20n, Perfect passives:C 0402 (1005 Metric), F.Cu at (163.0, 111.8)
- added Q201: SI8487DB, CSP-xxx:WLCSP-4 (1.56x1.56) P0.8, F.Cu at (118.5, 102.0)
- added Q202: 2N7002KNC, DFN-x:DFN-1006-3L, F.Cu at (123.0, 101.0)
- added R206: 100k, Perfect passives:R 0402 (1005 Metric), F.Cu at (162.2, 104.0)
- added R207: 100k, Perfect passives:R 0402 (1005 Metric), F.Cu at (147.0, 97.0)
- added R208: 100k, Perfect passives:R 0402 (1005 Metric), F.Cu at (145.2, 97.5)
- added R210: 100k, Perfect passives:R 0402 (1005 Metric), F.Cu at (162.2, 100.5)
- added SW202: GT-TC024A, Buttons SMD:GT-TC024A-H0060-L1, F.Cu at (163.2, 114.5)
- added SW501: MINI 12C02, Slide switch SMD:MINI MSK12CO2, B.Cu at (117.0, 113.8)
- added U1: ESP32-C3-MINI-1U, RF modules:ESP32-C3-MINI-1U, F.Cu at (153.5, 105.0)
- added U802: HUSB237, SON-xx:SON-6 (2x2) P0.65, F.Cu at (163.0, 108.8)
- C201, C801: value 1u -> 100n
- C313, C314: value 10u -> 22u
- C315: value 10u -> 100n; footprint Perfect passives:C 0805 (2012 Metric) -> Perfect passives:C 0402 (1005 Metric)
- C507: value 100u -> 47u
- D201: value LESD8D3.3CAT5G -> BN5A1V40; footprint DFN-x:DFN-1006-2L -> DFN-x:DFN1610-2L (1.6x1)
- D302: value LEDR -> CZRQC8V2B; footprint LED SMD:LED-0402-R -> DFN-x:DFN-1006-2L
- J201: value U.FL-R-SMT-1 -> A1257WR-S-2P; footprint RF connectors:U.FL-R-1 -> Connectors SMD:A1257WR-S-2P (GH); moved to B.Cu
- J901, J902, J903, J904, J905, J906: value FPC-0.5AL-12PB -> 1.0-9P LT (SH); footprint Connectors FFC SMD:FPC-0.5AL-12PB -> Connectors SMD:1.0-9P LT (SH)
- L501: footprint Inductors SMD:AAPS0660MxxxF -> Inductors THT:PDMTAT044125-220MWU; moved to B.Cu
- Q301: value 30P03D -> DOZ60P03
- R311: value 1k -> 100k
- U201: value ESP32-C3 -> TMP235; footprint QFN-x generic:QFN-32 (5x5) P0.5 ESP -> SOT-xxx:SOT-363-5
- U202: value ZD25WQ32C -> LMV331; footprint SON-xx:USON-8 (2x3) P0.5 -> SOT-xxx:SOT-363-5
- moved D201 47.1 mm to (116.5, 102.0), turned to -90 degrees
- moved J201 45.4 mm to (118.0, 103.5)
- moved D302 43.9 mm to (149.0, 76.2), turned to 45 degrees
- moved D101 42.8 mm to (161.0, 116.0), turned to 0 degrees
- moved R311 41.7 mm to (147.8, 76.0), turned to -135 degrees
- moved C102 41.3 mm to (158.2, 114.2)
- moved C101 41.2 mm to (161.2, 114.0)
- moved U101 41.2 mm to (159.8, 114.0)
- moved R201 41.2 mm to (123.0, 102.0)
- moved R101 38.8 mm to (158.8, 116.0), turned to 180 degrees
- moved R203 38.6 mm to (124.5, 99.5), turned to -90 degrees
- moved C315 36.6 mm to (160.0, 97.5)
- moved R204 36.1 mm to (124.5, 101.5), turned to 90 degrees
- moved R202 31.9 mm to (123.5, 99.5)
- moved R516 29.1 mm to (119.0, 114.2), turned to 180 degrees
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Connections:
- C201 pad 1: +3V3 -> /MCU/MCU.BOOT
- C315 pad 1: +5VLED -> +PVDD
- C801 pad 1: +VCH221 -> +VBUS
- D201 pad 1: /MCU/MCU.boot -> /MCU/+VFAN
- D302 pad 1: Net-(D302-K) -> +PVDD
- D302 pad 2: Net-(D302-A) -> /PSU/PVDD.PG
- J201 pad 1: Net-(J201-In) -> /MCU/+VFAN
- J901 pad 5: /LED CONNECTORS/-VLEDHP.1 -> +VLED
- J901 pad 6: +VLED -> /LED CONNECTORS/-VLEDCRI.1
- J901 pad 7: +VLED -> +HVLEDCRI
- J901 pad 8: /LED CONNECTORS/-VLEDCRI.1 -> +VLED
- J901 pad 9: unconnected-(J901-Pin_9-Pad9) -> /LED CONNECTORS/+VLEDR.1M2
- J902 pad 5: /LED CONNECTORS/-VLEDHP.2 -> +VLED
- J902 pad 6: +VLED -> /LED CONNECTORS/-VLEDCRI.2
- J902 pad 7: +VLED -> +HVLEDCRI
- J902 pad 8: /LED CONNECTORS/-VLEDCRI.2 -> /LED CONNECTORS/+VLEDR.1M2
- J902 pad 9: unconnected-(J902-Pin_9-Pad9) -> /LED CONNECTORS/-VLEDR.1
- J903 pad 5: /LED CONNECTORS/-VLEDHP.3 -> +VLED
- J903 pad 6: +VLED -> /LED CONNECTORS/-VLEDCRI.3
- J903 pad 7: +VLED -> +HVLEDCRI
- J903 pad 8: /LED CONNECTORS/-VLEDCRI.3 -> +VLED
- J903 pad 9: unconnected-(J903-Pin_9-Pad9) -> /LED CONNECTORS/+VLEDR.3M4
- J904 pad 5: /LED CONNECTORS/-VLEDHP.4 -> +VLED
- J904 pad 6: +VLED -> /LED CONNECTORS/-VLEDCRI.4
- J904 pad 7: +VLED -> +HVLEDCRI
- J904 pad 8: /LED CONNECTORS/-VLEDCRI.4 -> /LED CONNECTORS/+VLEDR.3M4
- J904 pad 9: unconnected-(J904-Pin_9-Pad9) -> /LED CONNECTORS/-VLEDR.2
- J905 pad 5: /LED CONNECTORS/-VLEDHP.5 -> +VLED
- J905 pad 6: +VLED -> /LED CONNECTORS/-VLEDCRI.5
- J905 pad 7: +VLED -> +HVLEDCRI
- J905 pad 8: /LED CONNECTORS/-VLEDCRI.5 -> +VLED
- J905 pad 9: unconnected-(J905-Pin_9-Pad9) -> /LED CONNECTORS/+VLEDR.5M6
- J906 pad 5: /LED CONNECTORS/-VLEDHP.6 -> +VLED
- J906 pad 6: +VLED -> /LED CONNECTORS/-VLEDCRI.6
- J906 pad 7: +VLED -> +HVLEDCRI
- J906 pad 8: /LED CONNECTORS/-VLEDCRI.6 -> /LED CONNECTORS/+VLEDR.5M6
- J906 pad 9: unconnected-(J906-Pin_9-Pad9) -> /LED CONNECTORS/-VLEDR.3
- Q402 pad 1: /LED DRIVERS/LED RED/LEDR.FLT -> /LED DRIVERS/LED CW HIGH POWER/LEDHP.FLT1
- R201 pad 1: /MCU/MCU.boot -> Net-(Q201-G)
- R201 pad 2: +3V3 -> +VLED
- R202 pad 1: /MCU/MCU.strap2 -> Net-(U202A-A-)
- R203 pad 1: /MCU/MCU.strap1 -> GND
- R203 pad 2: +3V3 -> Net-(U202A-A-)
- R204 pad 1: /MCU/MCU.CHIP.EN -> Net-(Q202-G)
- R306 pad 1: /PSU/VLED.ANLG.FB -> Net-(R306-Pad1)
- R306 pad 2: Net-(R306-Pad2) -> /PSU/VLED.ANLG.FB
- R309 pad 1: Net-(R306-Pad2) -> Net-(R306-Pad1)
- R311 pad 1: Net-(D302-A) -> /PSU/PVDD.PG
- R311 pad 2: +3V3 -> GND
- R702 pad 2: /LED DRIVERS/LED RED/LEDR.FLT -> /LED DRIVERS/LED CW HIGH POWER/LEDHP.FLT1
- U201 pad 1: /MCU/MCU.RF.LNAIN -> GND
- U201 pad 2: /MCU/+V3P3 -> GND
- U201 pad 3: /MCU/+V3P3 -> /MCU/TMP
- U201 pad 4: /LED DRIVERS/LEDCRI.I2C0.SCL -> +3V3
- U201 pad 5: /LED DRIVERS/LEDCRI.I2C0.SDA -> GND
- U202 pad 1: /MCU/MCU.SPI0.CS -> /MCU/TMP
- U202 pad 2: /MCU/MCU.SPI0.PICO -> GND
- U202 pad 3: /MCU/MCU.SPI0.WP -> Net-(U202A-A-)
- U202 pad 4: GND -> Net-(Q202-G)
- U202 pad 5: /MCU/MCU.SPI0.POCI -> +3V3
- U203 pad 4: /MCU/MCU.strap1 -> /MCU/MCU.USRLED
- U601 pad 12: /LED DRIVERS/LED RED/LEDR.FLT -> /LED DRIVERS/LED CW HIGH POWER/LEDHP.FLT1
Routing:
- net /MCU/MCU.WS28: track 115.9 -> 11.8 mm, vias 4 -> 2
- net +3V3: track 147.2 -> 67.5 mm, vias 21 -> 18
- net /PSU/PVDD.PG: track 78.6 -> 10.5 mm, vias 3 -> 0
- net +HVLEDCRI: track 21.8 -> 87.0 mm
- net /PSU/VLED.PG: track 95.8 -> 32.9 mm
- net GND: track 174.4 -> 127.7 mm, vias 314 -> 178
- net /MCU/MCU.strap1: track 43.0 -> 0.00 mm, vias 4 -> 0
- net /LED DRIVERS/LEDHP.EN: track 54.1 -> 97.1 mm
- net /MCU/MCU.boot: track 35.3 -> 0.00 mm, vias 2 -> 0
- net /LED DRIVERS/LEDHP.P.0: track 62.3 -> 94.6 mm
- net /MCU/MCU.BOOT: track 0.00 -> 29.5 mm, vias 0 -> 2
- net +VBUS: track 8.62 -> 35.7 mm, vias 0 -> 2
- net /MCU/MCU.U.d-: track 34.6 -> 59.5 mm, vias 4 -> 3
- net /MCU/MCU.U.d+: track 34.7 -> 59.4 mm, vias 5 -> 4
- net /LED DRIVERS/LEDCRI.P.0: track 43.7 -> 19.9 mm
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- removed copper zone on In1.Cu, net +HVLEDCRI
- removed copper zone on F.Cu, net /MCU/+V3P3
- removed copper zone on F.Cu, net /MCU/MCU.RF.LNAIN
- removed copper zone on F.Cu, net Net-(J201-In)
Other:
- board text removed: "CH221 PWR"
- board text removed: "PFSET ADJ"
