File: LEDCRI.kicad_sch (KiCad schematic)
At the start: 47 parts, among them Q501 SI8487DB, Q502 SI8487DB, Q503 BSC0805LS, U501 LP8866

Commit message: Add files via upload
Parts:
- removed JP502: Conn_02x03_Odd_Even, Connector_PinHeader_1.00mm:PinHeader_2x03_P1.00mm_Vertical, symbol Connector_Generic:Conn_02x03_Odd_Even
- removed R514: 11k, Perfect passives:R 0402 (1005 Metric), symbol Device:R_Small_US
- added C518, C520, C521, C522: 10u, Perfect passives:C 0805 (2012 Metric), symbol Device:C_Small
- added C519: 22u, Capacitor_SMD:C_1206_3216Metric, symbol Device:C_Small
- added SW501: MINI 12C02, Slide switch SMD:MINI MSK12CO2, symbol Slide switch:SPDT
- C507: value 100u -> 47u
- L501: footprint Inductors SMD:AAPS0660MxxxF -> Inductors THT:PDMTAT044125-220MWU
Connections:
- net +HVLEDCRI: now also C520.1, C521.1, C522.1
- net +VINSD: now also C518.1, C519.1
- net GND: now also C518.2, C519.2, C520.2, C521.2, C522.2, SW501.2 (COM)
- net at R516.2: now also SW501.3 (C2)
- net at R515.2: now also SW501.1 (C1)
Other:
- note added: ">1.25Ω"
- note added: "PDMTAT044125-220MWU"
- note added: "SPZ1HM470E08O00RA"
- note removed: ">250mΩ"
- note removed: "AAPS0660M220F"
- note removed: "HGC0805R5106K500NSLJ"
- note removed: "PH101M050E140B000"
- moved on the sheet: C503, C504, C505, C506, C507, C508, R507, R508, R515, R516, R521
