File: PSU.kicad_sch (KiCad schematic)
At the start: 69 parts, among them Q301 30P03D, Q302 2N7002KNC, Q303 2N7002KNC, Q304 2N7002KNC, Q306 2N7002KNC, U301 SIC431A, U302 DZDH0401DW, U303 AP62600, U304 SY8301, U306 LMV331

Commit message: Add files via upload
Parts:
- removed C316: 10u, Perfect passives:C 0805 (2012 Metric), symbol Device:C_Small
- removed D302: LEDR, LED SMD:LED-0402-R, symbol SMD LED:NCD0402R1
- removed D309: LESD8D3.3CAT5G, DFN-x:DFN-1006-2L, symbol TVS diodes bidirectional:LESD8D3.3CAT5G
- removed Q301: 30P03D, DFN-x:DFN-8 (3x3) 1EP, symbol Mosfets P-channel:30P03D
- removed Q302: 2N7002KNC, DFN-x:DFN-1006-3L, symbol Mosfet N-channel:2N7002KNC
- removed R321, R322: 121k, Perfect passives:R 0402 (1005 Metric), symbol Device:R_Small_US
- removed R324: 100k, Perfect passives:R 0402 (1005 Metric), symbol Device:R_Small_US
- removed R325: 6k, Perfect passives:R 0402 (1005 Metric), symbol Device:R_Small_US
- removed R327: 20k, Perfect passives:R 0402 (1005 Metric), symbol Device:R_Small_US
- removed U306: LMV331, SOT-xxx:SOT-363-5, symbol Comparators:LMV331DCK
- added D302: CZRQC8V2B, DFN-x:DFN-1006-2L, symbol Zener diodes:CZRQC8V2B-HF
- added Q301: DOZ60P03, DFN-x:DFN-8 (3x3) 1EP, symbol Mosfets P-channel:DOZ60P03
- C313, C314: value 10u -> 22u
- C315: value 10u -> 100n; footprint Perfect passives:C 0805 (2012 Metric) -> Perfect passives:C 0402 (1005 Metric)
- R311: value 1k -> 100k
Connections:
- net +3V3: no longer R311.2
- net +5VLED: no longer C315.1
- net +PVDD: now also C315.1, D302.1 (K), Q301.1 (S), Q301.2 (S), Q301.3 (S)
- net +VBUS: now also Q301.5 (D)
- net GND: now also R311.2
- net PVDD.PG: now also R311.1, D302.2 (A)
- net VLED.ANLG.FB: now also R306.2; no longer R306.1
- net at R308.1, U302.3 (BIAS): now also Q301.4 (G)
- net at R309.1: now also R306.1; no longer R306.2
Other:
- note added: "6.66A²×0.0145 = 0.643W"
- note added: "SA11CM470A19R55XXX"
- note removed: "Buck section"
- note removed: "CHECKS IF PVDD IS > 10V"
- note removed: "ECASD31E226M040KA0"
- note removed: "PVDD LED"
- note removed: "PVDD PG comparator"
- note removed: "VBUS present"
- moved on the sheet: C302, C303, C311, C312, C317, C318, C319, C320, C321, D301, D303, D304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
