File: USB+PD.kicad_sch (KiCad schematic)
At the start: 11 parts, among them J801 HC-TYPE-C-16P-026W, U801 CH221K

Commit message: Add files via upload
Parts:
- removed JP801: Jumper_2_Small_Open, Solder jumpers:Jumper-NO 2P (1.9x1.4), symbol Jumper:Jumper_2_Small_Open
- removed R801: 200k, Perfect passives:R 0402 (1005 Metric), symbol Device:R_Small_US
- removed R802: 1k, Perfect passives:R 0402 (1005 Metric), symbol Device:R_Small_US
- removed U801: CH221K, SOT-xxx:SOT-23-6, symbol USB PD controllers:CH221K
- added C803: 20n, Perfect passives:C 0402 (1005 Metric), symbol Device:C_Small
- added U802: HUSB237, SON-xx:SON-6 (2x2) P0.65, symbol USB PD controllers:HUSB237-AA001
- C801: value 1u -> 100n
- R803, R804: now not fitted
Connections:
- net +VCH221 is gone; now on net +VBUS: C801.1
- net +VBUS: now also U802.2 (VBUS)
- net CC1: now also U802.1 (CC1)
- net CC2: now also U802.6 (CC2)
- net GND: now also C803.2, U802.7 (GND)
- new net: C803.1, U802.3 (VSET)
- no-connect marks 6 -> 7
Other:
- note removed: "Power CH221K from 3V3"
- moved on the sheet: C801
